File: KiCad/mactxlc.kicad_pcb (KiCad board)
At the start: 2 copper layers, 54.8 x 36.8 mm, 8 parts, among them J1 Conn_02x12_Top_Bottom, J2 Conn_01x07, SW1 SW_DIP_x01, U1 MAX660

Commit message: Updated to KiCad 6 and silkscreen updates
Connections:
- net /-12 renamed /-5
- J1 pad 1: Net-(J1-Pad1) -> unconnected-(J1-Pad1)
- J1 pad 12: Net-(J1-Pad12) -> unconnected-(J1-Pad12)
- J1 pad 13: Net-(J1-Pad13) -> unconnected-(J1-Pad13)
- J1 pad 14: Net-(J1-Pad14) -> unconnected-(J1-Pad14)
- J1 pad 2: Net-(J1-Pad2) -> unconnected-(J1-Pad2)
- J1 pad 20: Net-(J1-Pad20) -> unconnected-(J1-Pad20)
- J1 pad 8: Net-(J1-Pad8) -> unconnected-(J1-Pad8)
- J1 pad 9: Net-(J1-Pad9) -> unconnected-(J1-Pad9)
- J2 pad 6: /+12 -> unconnected-(J2-Pad6)
- U1 pad 1: Net-(U1-Pad1) -> unconnected-(U1-Pad1)
- U1 pad 6: Net-(U1-Pad6) -> unconnected-(U1-Pad6)
- U1 pad 7: Net-(U1-Pad7) -> unconnected-(U1-Pad7)
Other:
- net class Default removed
- board text added: "+12"
- board text added: "+12v"
- board text added: "+3.3v"
- board text added: "+5v"
- board text added: "+5v STBY"
- board text added: "-12v"
- board text added: "GND"
- board text added: "NC"
- board text added: "PS-ON"
- board text added: "PWR GOOD"
- board text added: "Rev1.3"
- board text removed: "Rev1.2"
