File: mactx_lc_v2p0/mactxlc.kicad_sch (KiCad schematic)
At the start: 8 parts, among them J1 Conn_02x12_Top_Bottom, J2 Conn_01x07, SW1 SW_DIP_x01, U1 MAX660

Commit message: Fixed LC power connector and resistor part number
Parts:
- added D1: LED_Small, LED_SMD:LED_0805_2012Metric, symbol Device:LED_Small
- added JP1: SolderJumper_2_Open, Jumper:SolderJumper-2_P1.3mm_Open_RoundedPad1.0x1.5mm, symbol Jumper:SolderJumper_2_Open
- added R3: 10k, Resistor_SMD:R_0805_2012Metric, symbol Device:R
- J2: footprint Connector_TE-Connectivity:TE_826576-7_1x07_P3.96mm_Vertical -> Connector_Molex:Molex_KK-396_A-41791-0007_1x07_P3.96mm_Vertical
- R1, R2: LCSC C17903 -> C17414
Connections:
- net +5: now also JP1.2 (B)
- net GND: now also D1.1 (K)
- new net: JP1.1 (A), R3.2
- new net: D1.2 (A), R3.1
Changed lines of the file:
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@@
+    (stroke (width 0) (type default) (color 0 0 0 0))
+  )
+  (wire (pts (xy 134.62 78.74) (xy 134.62 86.36))
     (stroke (width 0) (type default) (color 0 0 0 0))
   )
@@
     (stroke (width 0) (type default) (color 0 0 0 0))
   )
+  (wire (pts (xy 134.62 66.04) (xy 134.62 71.12))
+    (stroke (width 0) (type default) (color 0 0 0 0))
+  )
   (wire (pts (xy 68.58 71.12) (xy 69.85 71.12))
     (stroke (width 0) (type default) (color 0 0 0 0))
   )
+  (wire (pts (xy 134.62 101.6) (xy 134.62 107.95))
+    (stroke (width 0) (type default) (color 0 0 0 0))
+  )
   (wire (pts (xy 68.58 60.96) (xy 73.66 60.96))
     (stroke (width 0) (type default) (color 0 0 0 0))
@@
     (stroke (width 0) (type default) (color 0 0 0 0))
   )
+  (wire (pts (xy 134.62 93.98) (xy 134.62 96.52))
+    (stroke (width 0) (type default) (color 0 0 0 0))
+  )
   (wire (pts (xy 85.09 76.2) (xy 85.09 53.34))
     (stroke (width 0) (type default) (color 0 0 0 0))
@@
     (stroke (width 0) (type default) (color 0 0 0 0))
   )
+  (label "+5" (at 134.62 68.58 90)
+    (effects (font (size 1.27 1.27)) (justify left bottom))
+  )
   (label "GND" (at 93.98 53.34 0)
+    (effects (font (size 1.27 1.27)) (justify left bottom))
+  )
+  (label "GND" (at 134.62 107.95 90)
     (effects (font (size 1.27 1.27)) (justify left bottom))
   )
@@
       (effects (font (size 1.27 1.27)) (justify left))
     )
-    (property "Footprint" "Connector_TE-Connectivity:TE_826576-7_1x07_P3.96mm_Vertical" (id 2) (at 124.46 58.42 0)
+    (property "Footprint" "Connector_Molex:Molex_KK-396_A-41791-0007_1x07_P3.96mm_Vertical" (id 2) (at 124.46 58.42 0)
       (effects (font (size 1.27 1.27)) hide)
     )
@@
       (effects (font (size 1.27 1.27)) hide)
     )
-    (property "LCSC" "C17903" (id 4) (at 69.85 97.79 0)
+    (property "LCSC" "C17414" (id 4) (at 69.85 97.79 0)
       (effects (font (size 1.27 1.27)) hide)
     )
@@
       (effects (font (size 1.27 1.27)) hide)
     )
-    (property "LCSC" "C17903" (id 4) (at 60.96 111.76 0)
+    (property "LCSC" "C17414" (id 4) (at 60.96 111.76 0)
+      (effects (font (size 1.27 1.27)) hide)
+    )
+    (pin "1")
+    (pin "2")
+  )
+  (symbol (lib_id "Jumper:SolderJumper_2_Open") (at 134.62 74.93 90) (unit 1)
+    (in_bom yes) (on_board yes) (fields_autoplaced)
+    (property "Reference" "JP1" (id 0) (at 137.16 73.6599 90)
+      (effects (font (size 1.27 1.27)) (justify right))
+    )
+    (property "Value" "SolderJumper_2_Open" (id 1) (at 137.16 76.1999 90)
+      (effects (font (size 1.27 1.27)) (justify right))
+    )
+    (property "Footprint" "Jumper:SolderJumper-2_P1.3mm_Open_RoundedPad1.0x1.5mm" (id 2) (at 134.62 74.93 0)
+      (effects (font (size 1.27 1.27)) hide)
+    )
+    (property "Datasheet" "~" (id 3) (at 134.62 74.93 0)
+      (effects (font (size 1.27 1.27)) hide)
+    )
+    (pin "1")
+    (pin "2")
+  )
+  (symbol (lib_id "Device:R") (at 134.62 90.17 180) (unit 1)
+    (in_bom yes) (on_board yes)
+    (property "Reference" "R3" (id 0) (at 138.43 91.44 0)
+      (effects (font (size 1.27 1.27)) (justify left))
+    )
+    (property "Value" "10k" (id 1) (at 139.7 88.9 0)
+      (effects (font (size 1.27 1.27)) (justify left))
+    )
+    (property "Footprint" "Resistor_SMD:R_0805_2012Metric" (id 2) (at 136.398 90.17 90)
+      (effects (font (size 1.27 1.27)) hide)
+    )
+    (property "Datasheet" "~" (id 3) (at 134.62 90.17 0)
+      (effects (font (size 1.27 1.27)) hide)
+    )
+    (property "LCSC" "C17414" (id 4) (at 134.62 90.17 0)
+      (effects (font (size 1.27 1.27)) hide)
+    )
+    (pin "1")
+    (pin "2")
+  )
+  (symbol (lib_id "Device:LED_Small") (at 134.62 99.06 90) (unit 1)
+    (in_bom yes) (on_board yes) (fields_autoplaced)
+    (property "Reference" "D1" (id 0) (at 137.16 97.7264 90)
+      (effects (font (size 1.27 1.27)) (justify right))
+    )
+    (property "Value" "LED_Small" (id 1) (at 137.16 100.2664 90)
+      (effects (font (size 1.27 1.27)) (justify right))
+    )
+    (property "Footprint" "LED_SMD:LED_0805_2012Metric" (id 2) (at 134.62 99.06 90)
+      (effects (font (size 1.27 1.27)) hide)
+    )
+    (property "Datasheet" "~" (id 3) (at 134.62 99.06 90)
+      (effects (font (size 1.27 1.27)) hide)
+    )
+    (property "LCSC" "C2297" (id 4) (at 134.62 99.06 90)
       (effects (font (size 1.27 1.27)) hide)
     )
@@
       (reference "C2") (unit 1) (value "10uf") (footprint "Capacitor_SMD:C_Elec_4x5.4")
     )
+    (path "/c78a3bed-31a5-4d1a-b29f-ade0b09bdb1f"
+      (reference "D1") (unit 1) (value "LED_Small") (footprint "LED_SMD:LED_0805_2012Metric")
+    )
     (path "/00000000-0000-0000-0000-00005df5f6f9"
       (reference "J1") (unit 1) (value "Conn_02x12_Top_Bottom") (footprint "Connector_Molex:Molex_Mini-Fit_Jr_5566-24A_2x12_P4.20mm_Vertical")
     )
     (path "/00000000-0000-0000-0000-00005df63ba9"
-      (reference "J2") (unit 1) (value "Conn_01x07") (footprint "Connector_TE-Connectivity:TE_826576-7_1x07_P3.96mm_Vertical")
+      (reference "J2") (unit 1) (value "Conn_01x07") (footprint "Connector_Molex:Molex_KK-396_A-41791-0007_1x07_P3.96mm_Vertical")
+    )
+    (path "/1dee33d7-3a8f-4877-ba94-3056a29b21d0"
+      (reference "JP1") (unit 1) (value "SolderJumper_2_Open") (footprint "Jumper:SolderJumper-2_P1.3mm_Open_RoundedPad1.0x1.5mm")
     )
     (path "/00000000-0000-0000-0000-00005e0ab748"
@@
       (reference "R2") (unit 1) (value "10k") (footprint "Resistor_SMD:R_0805_2012Metric")
     )
+    (path "/4e7277b8-8a25-4181-95e8-e09bd3dcd4ba"
+      (reference "R3") (unit 1) (value "10k") (footprint "Resistor_SMD:R_0805_2012Metric")
+    )
     (path "/00000000-0000-0000-0000-00005df71407"
